File: hardware/main.sch (EAGLE design)
At the start: 60 parts, among them CON1 WIRE2BOARD_10POS, CON2 WIRE2BOARD_10POS, U1 SN74LVC4245A_DW_24, U2 Value, U3 SN74ABT541B_DW_20, U4 SN74LVC1G04_DBV_5, U5 SN74LVC4245A_DW_24, U6 Value, U7 TXB0101_DBV_6, U8 8BIT-DIP-SWITCH, U9 LM3940SOT223

Commit message: Cleaned up board. Cleaned up schematic. No structural or electrical changes
Other:
- moved on the sheet: C2
Changed lines of the file:
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@@
 <wire x1="172.72" y1="297.18" x2="172.72" y2="177.8" width="0.1524" layer="97"/>
 <wire x1="259.08" y1="58.42" x2="271.78" y2="58.42" width="0.1524" layer="97"/>
-<wire x1="271.78" y1="58.42" x2="307.34" y2="58.42" width="0.1524" layer="97"/>
-<wire x1="307.34" y1="58.42" x2="327.66" y2="58.42" width="0.1524" layer="97"/>
-<wire x1="327.66" y1="58.42" x2="474.98" y2="58.42" width="0.1524" layer="97"/>
+<wire x1="271.78" y1="58.42" x2="474.98" y2="58.42" width="0.1524" layer="97"/>
 <wire x1="474.98" y1="58.42" x2="474.98" y2="177.8" width="0.1524" layer="97"/>
 <wire x1="474.98" y1="177.8" x2="332.74" y2="177.8" width="0.1524" layer="97"/>
@@
 <text x="261.62" y="261.62" size="2.54" layer="97">OUTPUT PERIPHERALS</text>
 <wire x1="137.16" y1="0" x2="271.78" y2="0" width="0.1524" layer="97"/>
-<wire x1="271.78" y1="0" x2="271.78" y2="45.72" width="0.1524" layer="97"/>
-<wire x1="271.78" y1="45.72" x2="271.78" y2="58.42" width="0.1524" layer="97"/>
+<wire x1="271.78" y1="0" x2="271.78" y2="58.42" width="0.1524" layer="97"/>
 <wire x1="137.16" y1="45.72" x2="165.1" y2="45.72" width="0.1524" layer="97"/>
 <wire x1="165.1" y1="45.72" x2="165.1" y2="58.42" width="0.1524" layer="97"/>
@@
 <instance part="GND16" gate="1" x="325.12" y="147.32"/>
 <instance part="C1" gate="G$1" x="314.96" y="154.94"/>
-<instance part="C2" gate="G$1" x="406.4" y="162.56" rot="R90"/>
-<instance part="GND17" gate="1" x="411.48" y="157.48"/>
+<instance part="C2" gate="G$1" x="411.48" y="157.48"/>
+<instance part="GND17" gate="1" x="411.48" y="147.32"/>
 <instance part="R17" gate="G$1" x="292.1" y="243.84" rot="R180"/>
 <instance part="D9" gate="G$1" x="304.8" y="243.84" rot="R270"/>
@@
 <wire x1="393.7" y1="154.94" x2="396.24" y2="154.94" width="0.1524" layer="91"/>
 <pinref part="C2" gate="G$1" pin="1"/>
-<wire x1="401.32" y1="162.56" x2="396.24" y2="162.56" width="0.1524" layer="91"/>
+<wire x1="411.48" y1="162.56" x2="396.24" y2="162.56" width="0.1524" layer="91"/>
 <junction x="396.24" y="162.56"/>
 </segment>
@@
 <pinref part="C2" gate="G$1" pin="2"/>
 <pinref part="GND17" gate="1" pin="GND"/>
-<wire x1="408.94" y1="162.56" x2="411.48" y2="162.56" width="0.1524" layer="91"/>
-<wire x1="411.48" y1="162.56" x2="411.48" y2="160.02" width="0.1524" layer="91"/>
-</segment>
-<segment>
+<wire x1="411.48" y1="154.94" x2="411.48" y2="149.86" width="0.1524" layer="91"/>
+</segment>
+<segment>

Commit message: Added pulldown resistors on inputs. Updated version number
Parts:
- added R26, R27, R28, R29, R30, R31, R32, R33, R34, R35, R36, R37, R38, R39, R40, R41: 10k, SparkFun-Resistors:RESISTOR0805-RES
Connections:
- net GND: now also R26.1, R27.1, R28.1, R29.1, R30.1, R31.1, R32.1, R33.1, R34.1, R35.1, R36.1, R37.1, R38.1, R39.1, R40.1, R41.1
- net N$1: now also R29.2
- net N$2: now also R28.2
- net N$3: now also R27.2
- net N$4: now also R26.2
- net N$5: now also R30.2
- net N$6: now also R31.2
- net N$7: now also R32.2
- net N$8: now also R33.2
- net UCOUT1: now also R41.2
- net UCOUT2: now also R40.2
- net UCOUT3: now also R39.2
- net UCOUT4: now also R38.2
- net UCOUT5: now also R37.2
- net UCOUT6: now also R36.2
- net UCOUT7: now also R35.2
- net UCOUT8: now also R34.2
Other:
- moved on the sheet: C1, C2, D10, D11, D12, D13, D14, D15, D16, D9, R17, R18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

Commit message: Re-routed and updated board and schematic
Parts:
- removed C1, C2: 0.1uF, SparkFun-Capacitors:1.0UF-25V-+80/-20(0805)
- removed CON1, CON2: WIRE2BOARD_10POS, ControllerCard:WIRE2BOARD_10POS
- removed R1, R2, R26, R27, R28, R29, R3, R30, R31, R32, R33, R34, R35, R36, R37, R38, R39, R4, R40, R41, R5, R6, R7, R8: 10k, SparkFun-Resistors:RESISTOR0805-RES
- removed U2, U6: Value, ControllerCard:SN64BCT25244DW
- removed U3: SN74ABT541B_DW_20, ControllerCard:SN74ABT541B_DW_20
- removed U4: SN74LVC1G04_DBV_5, ControllerCard:SN74LVC1G04_DBV_5
- removed U7: TXB0101_DBV_6, ControllerCard:TXB0101_DBV_6
- removed U8: 8BIT-DIP-SWITCH, ControllerCard:8BIT-DIP-SWITCH
- added U$1, U$3, U$4: 4PIN_SOCKET, ControllerCard:4PIN_SOCKET
- added U$5, U$6: 2PIN_SOCKET, ControllerCard:2PIN_SOCKET
- added U$7, U$8: RESISTOR_ARRAY, ControllerCard:RESISTOR_ARRAY
- R10, R11, R12, R13, R14, R15, R16, R9: value 300 -> 330
- R25: value 300 -> 4.7k
- U$2: value M2-SWITCH -> 4PIN_SOCKET; device ControllerCard:M2-SWITCH -> ControllerCard:4PIN_SOCKET
Connections:
- removed net !INSEL!: U2.1OE_N, U2.2OE_N, U4.Y
- removed net !OUTBUFEN!: U6.1OE_N, U6.2OE_N, U7.B
- removed net INSEL: U$2.OUT2, U3.*OE1, U3.*OE2, U4.A
- removed net LEDIN1: D1.A, U1.A1, U2.1Y1, U3.Y8
- removed net LEDIN2: D2.A, U1.A2, U2.1Y2, U3.Y7
- removed net LEDIN3: D3.A, U1.A3, U2.1Y3, U3.Y6
- removed net LEDIN4: D4.A, U1.A4, U2.1Y4, U3.Y5
- removed net LEDIN5: D5.A, U1.A5, U2.2Y1, U3.Y4
- removed net LEDIN6: D6.A, U1.A6, U2.2Y2, U3.Y3
- removed net LEDIN7: D7.A, U1.A7, U2.2Y3, U3.Y2
- removed net LEDIN8: D8.A, U1.A8, U2.2Y4, U3.Y1
- removed net LEDOUT1: D9.A, U5.A1, U6.1Y1
- removed net LEDOUT2: D10.A, U5.A2, U6.1Y2
- removed net LEDOUT3: D11.A, U5.A3, U6.1Y3
- removed net LEDOUT4: D12.A, U5.A4, U6.1Y4
- removed net LEDOUT5: D13.A, U5.A5, U6.2Y1
- removed net LEDOUT6: D14.A, U5.A6, U6.2Y2
- removed net LEDOUT7: D15.A, U5.A7, U6.2Y3
- removed net LEDOUT8: D16.A, U5.A8, U6.2Y4
- removed net SW1: R1.2, U3.A8, U8.IN1
- removed net SW2: R2.2, U3.A7, U8.IN2
- removed net SW3: R3.2, U3.A6, U8.IN3
- removed net SW4: R4.2, U3.A5, U8.IN4
- removed net SW5: R5.2, U3.A4, U8.IN5
- removed net SW6: R6.2, U3.A3, U8.IN6
- removed net SW7: R7.2, U3.A2, U8.IN7
- removed net SW8: R8.2, U3.A1, U8.IN8
- net !BUFEN!: now also A1.P$18; no longer A1.P$38, U7.A
- net 3.3V: now also R25.1; no longer C1.1, U7.VCCA
- net 5V: now also U$5.P1, U$6.P1; no longer A1.P$21, C2.1, CON1.10, CON2.10, R25.1, U$2.IN1, U2.VCC, U2.VCC_2, U3.VCC, U4.VCC, U6.VCC, U6.VCC_2, U7.VCCB, U8.CL1, U8.CL2, U8.CL3, U8.CL4, U8.CL5, U8.CL6, U8.CL7, U8.CL8
- net ENEXT: no longer U7.OE
- net GND: now also U$5.P2, U$6.P2, U$7.1B, U$7.2B, U$7.3B, U$7.4B, U$7.5B, U$7.6B, U$7.7B, U$7.8B, U$8.1B, U$8.2B, U$8.3B, U$8.4B, U$8.5B, U$8.6B, U$8.7B, U$8.8B; no longer C1.2, C2.2, CON1.1, CON2.1, R1.1, R2.1, R26.1, R27.1, R28.1, R29.1, R3.1, R30.1, R31.1, R32.1, R33.1, R34.1, R35.1, R36.1, R37.1, R38.1, R39.1, R4.1, R40.1, R41.1, R5.1, R6.1, R7.1, R8.1, U$2.IN3, U2.GND, U2.GND_2, U2.GND_3, U2.GND_4, U3.GND, U4.GND, U6.GND, U6.GND_2, U6.GND_3, U6.GND_4, U7.GND
- net N$1: now also U$1.P1, U$7.1A, U1.A8; no longer CON1.5, R29.2, U2.2A1
- net N$17: now also U$4.P1, U5.A1; no longer CON2.5, U6.2A1
- net N$18: now also U$4.P2, U5.A2; no longer CON2.4, U6.2A2
- net N$19: now also U$4.P3, U5.A3; no longer CON2.3, U6.2A3
- net N$2: now also U$1.P2, U$7.2A, U1.A7; no longer CON1.4, R28.2, U2.2A2
- net N$20: now also U$4.P4, U5.A4; no longer CON2.2, U6.2A4
- net N$21: now also U$2.P1, U5.A5; no longer CON2.6, U6.1A4
- net N$22: now also U$2.P2, U5.A6; no longer CON2.7, U6.1A3
- net N$23: now also U$2.P3, U5.A7; no longer CON2.8, U6.1A2
- net N$24: now also U$2.P4, U5.A8; no longer CON2.9, U6.1A1
- net N$3: now also U$1.P3, U$7.3A, U1.A6; no longer CON1.3, R27.2, U2.2A3
- net N$4: now also U$1.P4, U$7.4A, U1.A5; no longer CON1.2, R26.2, U2.2A4
- net N$5: now also U$3.P1, U$7.5A, U1.A4; no longer CON1.6, R30.2, U2.1A4
- net N$6: now also U$3.P2, U$7.6A, U1.A3; no longer CON1.7, R31.2, U2.1A3
- net N$7: now also U$3.P3, U$7.7A, U1.A2; no longer CON1.8, R32.2, U2.1A2
- net N$8: now also U$3.P4, U$7.8A, U1.A1; no longer CON1.9, R33.2, U2.1A1
- net UCIN1: now also A1.P$19, D1.A; no longer A1.P$39
- net UCIN2: now also A1.P$40, D2.A; no longer A1.P$19
- net UCIN3: now also A1.P$39, D3.A; no longer A1.P$40
- net UCIN4: now also A1.P$5, D4.A; no longer A1.P$10
- net UCIN5: now also A1.P$7, D5.A; no longer A1.P$9
- net UCIN6: now also D6.A
- net UCIN7: now also A1.P$9, D7.A; no longer A1.P$7
- net UCIN8: now also A1.P$10, D8.A; no longer A1.P$5
- net UCOUT1: now also A1.P$38, D9.A, U$8.1A; no longer A1.P$18, R41.2
- net UCOUT2: now also D10.A, U$8.2A; no longer R40.2
- net UCOUT3: now also D11.A, U$8.3A; no longer R39.2
- net UCOUT4: now also D12.A, U$8.4A; no longer R38.2
- net UCOUT5: now also D13.A, U$8.5A; no longer R37.2
- net UCOUT6: now also D14.A, U$8.6A; no longer R36.2
- net UCOUT7: now also D15.A, U$8.7A; no longer R35.2
- net UCOUT8: now also D16.A, U$8.8A; no longer R34.2
Other:
- note removed: "INPUT PERIPHERALS"
- note removed: "OUTPUT PERIPHERALS"
- moved on the sheet: D1, D10, D11, D12, D13, D14, D15, D16, D17, D2, D3, D4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

Commit message: Updated with DRC modifications
Parts:
- renumbered U$7 to U7, U$8 to U8

Commit message: Minor component value changes. Added a BOM
Parts:
- R17, R18, R19, R20, R21, R22, R23, R24: value 300 -> 330
- R25: value 4.7k -> 330
Changed lines of the file:
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@@
 <part name="GND12" library="SparkFun-Aesthetics" deviceset="GND" device=""/>
 <part name="GND13" library="SparkFun-Aesthetics" deviceset="GND" device=""/>
-<part name="R17" library="SparkFun-Resistors" deviceset="RESISTOR" device="0805-RES" value="300"/>
+<part name="R17" library="SparkFun-Resistors" deviceset="RESISTOR" device="0805-RES" value="330"/>
 <part name="D9" library="SparkFun-LED" deviceset="LED" device="3MM"/>
 <part name="D10" library="SparkFun-LED" deviceset="LED" device="3MM"/>
@@
 <part name="D15" library="SparkFun-LED" deviceset="LED" device="3MM"/>
 <part name="D16" library="SparkFun-LED" deviceset="LED" device="3MM"/>
-<part name="R18" library="SparkFun-Resistors" deviceset="RESISTOR" device="0805-RES" value="300"/>
-<part name="R19" library="SparkFun-Resistors" deviceset="RESISTOR" device="0805-RES" value="300"/>
-<part name="R20" library="SparkFun-Resistors" deviceset="RESISTOR" device="0805-RES" value="300"/>
-<part name="R21" library="SparkFun-Resistors" deviceset="RESISTOR" device="0805-RES" value="300"/>
-<part name="R22" library="SparkFun-Resistors" deviceset="RESISTOR" device="0805-RES" value="300"/>
-<part name="R23" library="SparkFun-Resistors" deviceset="RESISTOR" device="0805-RES" value="300"/>
-<part name="R24" library="SparkFun-Resistors" deviceset="RESISTOR" device="0805-RES" value="300"/>
+<part name="R18" library="SparkFun-Resistors" deviceset="RESISTOR" device="0805-RES" value="330"/>
+<part name="R19" library="SparkFun-Resistors" deviceset="RESISTOR" device="0805-RES" value="330"/>
+<part name="R20" library="SparkFun-Resistors" deviceset="RESISTOR" device="0805-RES" value="330"/>
+<part name="R21" library="SparkFun-Resistors" deviceset="RESISTOR" device="0805-RES" value="330"/>
+<part name="R22" library="SparkFun-Resistors" deviceset="RESISTOR" device="0805-RES" value="330"/>
+<part name="R23" library="SparkFun-Resistors" deviceset="RESISTOR" device="0805-RES" value="330"/>
+<part name="R24" library="SparkFun-Resistors" deviceset="RESISTOR" device="0805-RES" value="330"/>
 <part name="GND18" library="SparkFun-Aesthetics" deviceset="GND" device=""/>
 <part name="JP1" library="SparkFun-Connectors" deviceset="POWER_JACK" device="SMD" value="5.5x2.1mm Barrel"/>
@@
 <part name="C4" library="SparkFun-Capacitors" deviceset="1.0UF-25V-+80/-20(0805)" device="" value="0.47uF"/>
 <part name="D17" library="SparkFun-LED" deviceset="LED" device="3MM"/>
-<part name="R25" library="SparkFun-Resistors" deviceset="RESISTOR" device="0805-RES" value="4.7k"/>
+<part name="R25" library="SparkFun-Resistors" deviceset="RESISTOR" device="0805-RES" value="330"/>
 <part name="GND20" library="SparkFun-Aesthetics" deviceset="GND" device=""/>
 <part name="GND22" library="SparkFun-Aesthetics" deviceset="GND" device=""/>

Commit message: Removed 'ENEXT', as it is not needed
Connections:
- removed net ENEXT: A1.P$36
Changed lines of the file:
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@@
-</segment>
-</net>
-<net name="ENEXT" class="0">
-<segment>
-<pinref part="A1" gate="G$1" pin="P$36"/>
-<wire x1="71.12" y1="25.4" x2="73.66" y2="25.4" width="0.1524" layer="91"/>
-<label x="73.66" y="25.4" size="1.016" layer="95" xref="yes"/>
 </segment>
 </net>
